Commit message: suction_cup and rgb-d camera

File: ur_description/urdf/inc/ur5_macro.xacro (robot description, xacro)
@@ -1,21 +1,21 @@
 <?xml version="1.0"?>
 <robot xmlns:xacro="http://wiki.ros.org/xacro">
-  <!--
-    Convenience wrapper for the 'ur_robot' macro which provides default values
-    for the various "parameters files" parameters for a UR5.
-    This file can be used when composing a more complex scene with one or more
-    UR5 robots.
-    While the generic 'ur_robot' macro could also be used, it would require
-    the user to provide values for all parameters, as that macro does not set
-    any model-specific defaults (not even for the generic parameters, such as
-    the visual and physical parameters and joint limits).
-    Refer to the main 'ur_macro.xacro' in this package for information about
-    use, contributors and limitations.
-    NOTE: users will most likely want to override *at least* the
-          'kinematics_parameters_file' parameter. Otherwise, a default kinematic
-          model will be used, which will almost certainly not correspond to any
-          real robot.
-  -->
-  <xacro:macro name="ur5_robot" params="
+    <!--
+      Convenience wrapper for the 'ur_robot' macro which provides default values
+      for the various "parameters files" parameters for a UR5.
+      This file can be used when composing a more complex scene with one or more
+      UR5 robots.
+      While the generic 'ur_robot' macro could also be used, it would require
+      the user to provide values for all parameters, as that macro does not set
+      any model-specific defaults (not even for the generic parameters, such as
+      the visual and physical parameters and joint limits).
+      Refer to the main 'ur_macro.xacro' in this package for information about
+      use, contributors and limitations.
+      NOTE: users will most likely want to override *at least* the
+            'kinematics_parameters_file' parameter. Otherwise, a default kinematic
+            model will be used, which will almost certainly not correspond to any
+            real robot.
+    -->
+    <xacro:macro name="ur5_robot" params="
    prefix
    joint_limits_parameters_file:='$(find ur_description)/config/ur5/joint_limits.yaml'
@@ -27,17 +27,19 @@
    safety_pos_margin:=0.15
    safety_k_position:=20"
-  >
-    <xacro:include filename="$(find ur_description)/urdf/inc/ur_macro.xacro"/>
-    <xacro:ur_robot
-      prefix="${prefix}"
-      joint_limits_parameters_file="${joint_limits_parameters_file}"
-      kinematics_parameters_file="${kinematics_parameters_file}"
-      physical_parameters_file="${physical_parameters_file}"
-      visual_parameters_file="${visual_parameters_file}"
-      transmission_hw_interface="${transmission_hw_interface}"
-      safety_limits="${safety_limits}"
-      safety_pos_margin="${safety_pos_margin}"
-      safety_k_position="${safety_k_position}"
-    />
-  </xacro:macro>
+    >
+        <xacro:include filename="$(find ur_description)/urdf/inc/ur_macro.xacro"/>
+        <xacro:ur_robot
+                prefix="${prefix}"
+                joint_limits_parameters_file="${joint_limits_parameters_file}"
+                kinematics_parameters_file="${kinematics_parameters_file}"
+                physical_parameters_file="${physical_parameters_file}"
+                visual_parameters_file="${visual_parameters_file}"
+                transmission_hw_interface="${transmission_hw_interface}"
+                safety_limits="${safety_limits}"
+                safety_pos_margin="${safety_pos_margin}"
+                safety_k_position="${safety_k_position}"
+        />
+        <xacro:include filename="$(find bin_picking)/urdf/camera.xacro"/>
+        <xacro:include filename="$(find bin_picking)/urdf/suction_cup.xacro"/>
+    </xacro:macro>
 </robot>

Commit message: small updates
+ limitations for better planning

File: ur_description/urdf/inc/ur5_macro.xacro (robot description, xacro)
@@ -40,6 +40,4 @@
                 safety_k_position="${safety_k_position}"
         />
-        <xacro:include filename="$(find bin_picking)/urdf/camera.xacro"/>
-        <xacro:include filename="$(find bin_picking)/urdf/suction_cup.xacro"/>
     </xacro:macro>
 </robot>

File: ur_description/urdf/ur5.xacro (robot description, xacro)
@@ -1,18 +1,26 @@
 <?xml version="1.0"?>
 <robot xmlns:xacro="http://wiki.ros.org/xacro" name="ur5_robot">
-  <!--
-    This is a convenience top-level xacro which loads the macro for the UR5e
-    which defines the default values for the various "parameters files"
-    parameters for a UR5e.
-    This file is only useful when loading a stand-alone, completely isolated
-    robot with only default values for all parameters such as the kinematics,
-    visual and physical parameters and joint limits.
-    This file is not intended to be integrated into a larger scene or other
-    composite xacro.
-    Instead, xacro:include 'inc/ur5e_macro.xacro' and override the defaults
-    for the arguments to that macro.
-    Refer to 'inc/ur_macro.xacro' for more information.
-  -->
-  <xacro:include filename="$(find ur_description)/urdf/inc/ur5_macro.xacro"/>
-  <xacro:ur5_robot prefix="" />
+    <!--
+      This is a convenience top-level xacro which loads the macro for the UR5e
+      which defines the default values for the various "parameters files"
+      parameters for a UR5e.
+      This file is only useful when loading a stand-alone, completely isolated
+      robot with only default values for all parameters such as the kinematics,
+      visual and physical parameters and joint limits.
+      This file is not intended to be integrated into a larger scene or other
+      composite xacro.
+      Instead, xacro:include 'inc/ur5e_macro.xacro' and override the defaults
+      for the arguments to that macro.
+      Refer to 'inc/ur_macro.xacro' for more information.
+    -->
+    <xacro:include filename="$(find ur_description)/urdf/inc/ur5_macro.xacro"/>
+    <xacro:ur5_robot prefix=""/>
+    <xacro:include filename="$(find bin_picking)/urdf/suction_cup.xacro"/>
+    <!-- world link -->
+    <link name="world"/>
+    <joint name="world_joint" type="fixed">
+      <parent link="world"/>
+      <child link="base_link"/>
+      <origin xyz="0 0 0" rpy="0 0 0"/>
+    </joint>
 </robot>

File: ur_gazebo/urdf/ur.xacro (robot description, xacro)
@@ -36,5 +36,5 @@
       - hardware_interface/EffortJointInterface
     NOTE: this value must correspond to the controller configured in the
-          controller .yaml files in the 'config' directory.
+          controller .yaml files in the 'config' directory.<link name="world"/>
   -->
   <xacro:arg name="transmission_hw_interface" default="hardware_interface/PositionJointInterface"/>

File: ur_gazebo/urdf/ur5_suction.xacro (robot description, xacro)
@@ -26,8 +26,8 @@
     <xacro:include filename="$(find ur_gazebo)/urdf/ur_macro.xacro"/>
     <!--Declare arguments -->
-    <xacro:arg name="joint_limit_params" default=""/>
-    <xacro:arg name="physical_params" default=""/>
-    <xacro:arg name="kinematics_params" default=""/>
-    <xacro:arg name="visual_params" default=""/>
+    <xacro:arg name="joint_limit_params" default='$(find ur_description)/config/ur5/joint_limits.yaml'/>
+    <xacro:arg name="physical_params" default="$(find ur_description)/config/ur5/physical_parameters.yaml"/>
+    <xacro:arg name="kinematics_params" default="$(find ur_description)/config/ur5/default_kinematics.yaml"/>
+    <xacro:arg name="visual_params" default="$(find ur_description)/config/ur5/visual_parameters.yaml"/>
     <!--
       legal values:
@@ -42,4 +42,5 @@
     <xacro:arg name="safety_pos_margin" default="0.15"/>
     <xacro:arg name="safety_k_position" default="20"/>
+    <xacro:arg name="spawn_z" default="0.0"/>
     <!-- Instantiate the Gazebo robot and pass it all the required arguments. -->
     <xacro:ur_robot_gazebo
@@ -65,7 +66,6 @@
         <parent link="world"/>
         <child link="base_link"/>
-        <origin xyz="0 0 0" rpy="0 0 0"/>
+        <origin xyz="0 0 $(arg spawn_z)" rpy="0 0 0"/>
     </joint>
-    <xacro:include filename="$(find bin_picking)/urdf/camera.xacro"/>
     <xacro:include filename="$(find bin_picking)/urdf/suction_cup.xacro"/>
 </robot>
